Commit message: Tool cylinder v1

File: KUKA_Task/ros_ws/src/iiwa_stack/iiwa_description/urdf/iiwa7.xacro (robot description, xacro)
@@ -85,5 +85,5 @@
       <parent link="${robot_name}_link_1"/>
       <child link="${robot_name}_link_2"/>
-      <origin xyz="0 0 0.19" rpy="${PI / 2}   0 ${PI}"/>
+      <origin xyz="0 0 0.19" rpy="${PI / 2}   ${-PI / 3} ${PI}"/>
       <axis xyz="0 0 1"/>
       <limit lower="${-120 * PI / 180}" upper="${120 * PI / 180}"
@@ -153,5 +153,5 @@
       <parent link="${robot_name}_link_3"/>
       <child link="${robot_name}_link_4"/>
-      <origin xyz="0 0 0.19" rpy="${PI / 2} 0 0"/>
+      <origin xyz="0 0 0.19" rpy="${PI / 2} ${PI / 6} 0"/>
       <axis xyz="0 0 1"/>
       <limit lower="${-120 * PI / 180}" upper="${120 * PI / 180}"
@@ -221,5 +221,5 @@
       <parent link="${robot_name}_link_5"/>
       <child link="${robot_name}_link_6"/>
-      <origin xyz="0 0.06070 0.19" rpy="${PI / 2} 0 0"/>
+      <origin xyz="0 0.06070 0.19" rpy="${PI / 2} ${-PI / 2} 0"/>
       <axis xyz="0 0 1"/>
       <limit lower="${-120 * PI / 180}" upper="${120 * PI / 180}"
