Commit message: shifted tool to another xacro

File: KUKA_Task/ros_ws/src/iiwa_stack_examples/iiwa_tool/iiwa_tool_description/urdf/iiwa_tool.urdf.xacro (robot description, xacro)
@@ -6,4 +6,6 @@
   <!--Import the iiwa7 macro -->
   <xacro:include filename="$(find iiwa_description)/urdf/iiwa7.xacro"/>
+  <!--Import the tool macro -->
+  <xacro:include filename="$(find iiwa_tool_description)/urdf/tool.xacro"/>
   <!--  Arguments for the iiwa7 macro  -->
   <xacro:arg name="hardware_interface" default="PositionJointInterface"/>
@@ -37,42 +39,7 @@
     <origin xyz="0 0 0" rpy="0 0 0"/>
   </xacro:iiwa7>
-  <!-- Tool properties -->
-  <property name="tool_mass" value="0.200" />
-  <property name="tool_joint_offset" value="0.00 0.00 0.00" />
-  <property name="tool_link_offset" value="0.00 0.00 0.5" />
-  <!--  Here we define a dummy joint between the tip of the iiwa7 and the base of the tool.
-  There is no offset between the two, that means the tool is attached at the robot flange. -->
-  <joint name="tool_joint" type="fixed">
-    <parent link="iiwa_link_ee" />
-    <child link = "tool_link" />
-    <origin xyz="${tool_joint_offset}" rpy="0 0 0" />
-  </joint>
-  <!-- Here we define the geometry of the tool. We designed the tool ourselves, so we have a mesh file that represents it.
-  Else, one can define it using a geometric representation that approximate it, like a cylinder (see commented lines) -->
-  <link name="tool_link">
-    <visual>
-      <origin xyz="0 0 0.15" rpy="0 0 0"/>
-      <geometry>
-	<!-- <mesh filename="package://iiwa_tool_description/meshes/visual/tool.stl"/> -->
-		<cylinder length="0.3" radius="0.00090"/>
-      </geometry>
-      <material name="Red"/>
-    </visual>
-    <collision>
-      <origin xyz="0 0 0.15" rpy="0 0 0"/>
-      <geometry>
-	<!-- <mesh filename="package://iiwa_tool_description/meshes/visual/tool.stl"/> -->
-		<cylinder length="0.3" radius="0.00090"/>
-      </geometry>
-      <material name="Red"/>
-    </collision>
-  </link>
-  <!--  Here we define another dummy joint. It is placed at the end of the tool, so we can then attach a frame at its TCP for control -->
-  <joint name="tool_tip_joint" type="fixed">
-    <parent link="tool_link" />
-    <child link = "tool_link_ee" />
-    <origin xyz="${tool_link_offset}" rpy="0 0 0" />
-  </joint>
-  <!--  The TCP frame is here defined -->
-  <link name="tool_link_ee"/>
+  <!-- Here we insert the tool attached to the robot end effector. -->
+  <xacro:tool parent="iiwa_link_ee">
+    <origin xyz="0 0 0" rpy="0 0 0"/>
+  </xacro:tool>
 </robot>

File: KUKA_Task/ros_ws/src/iiwa_stack_fishing/iiwa_description/urdf/iiwa7.xacro (robot description, xacro)
@@ -221,5 +221,5 @@
       <parent link="${robot_name}_link_5"/>
       <child link="${robot_name}_link_6"/>
-      <origin xyz="0 0.06070 0.19" rpy="${PI / 2} ${-PI / 2} 0"/>
+      <origin xyz="0 0.06070 0.19" rpy="${PI / 2} ${-PI / 3} 0"/>
       <axis xyz="0 0 1"/>
       <limit lower="${-120 * PI / 180}" upper="${120 * PI / 180}"

Commit message: pendulum sim v0.1

File: KUKA_Task/ros_ws/src/iiwa_stack_examples/iiwa_tool/iiwa_tool_description/urdf/iiwa_tool.urdf.xacro (robot description, xacro)
@@ -7,5 +7,5 @@
   <xacro:include filename="$(find iiwa_description)/urdf/iiwa7.xacro"/>
   <!--Import the tool macro -->
-  <xacro:include filename="$(find iiwa_tool_description)/urdf/tool.xacro"/>
+  <xacro:include filename="$(find iiwa_tool_description)/urdf/tool_pendulum.xacro"/>
   <!--  Arguments for the iiwa7 macro  -->
   <xacro:arg name="hardware_interface" default="PositionJointInterface"/>
@@ -40,6 +40,6 @@
   </xacro:iiwa7>
   <!-- Here we insert the tool attached to the robot end effector. -->
-  <xacro:tool parent="iiwa_link_ee">
+  <xacro:tool_pendulum parent="iiwa_link_ee">
     <origin xyz="0 0 0" rpy="0 0 0"/>
-  </xacro:tool>
+  </xacro:tool_pendulum>
 </robot>

File: KUKA_Task/ros_ws/src/iiwa_stack_fishing/iiwa_description/urdf/utilities.xacro (robot description, xacro)
@@ -6,15 +6,21 @@
   <!--Cuboid-->
   <xacro:macro name="cuboid_inertia" params="width height length mass">
-    <inertia ixx="${mass * (height * height + length * length) / 12)}"
-             iyy="${mass * (width * width + length * length) / 12)}"
-             izz="${mass * (width * width + height * height) / 12)}"
+    <inertia ixx="${mass * (height * height + length * length) / 12}"
+             iyy="${mass * (width * width + length * length) / 12}"
+             izz="${mass * (width * width + height * height) / 12}"
              ixy="0" iyz="0" ixz="0"/>
   </xacro:macro>
-  <!--Cylinder: length is along the y-axis! -->
+  <!--Cylinder: length is along the z-axis! -->
   <xacro:macro name="cylinder_inertia" params="radius length mass">
-    <inertia ixx="${mass * (3 * radius * radius + length * length) / 12)}"
-             iyy="${mass * radius* radius / 2)}"
-             izz="${mass * (3 * radius * radius + length * length) / 12)}"
+    <inertia ixx="${(mass * (3 * radius * radius + length * length)) / 12}"
+             iyy="${(mass * (3 * radius * radius + length * length)) / 12}"
+             izz="${(mass * radius* radius) / 2}"
              ixy="0" iyz="0" ixz="0"/>
   </xacro:macro>
+  <!--Sphere -->
+  <xacro:macro name="sphere_inertia" params="radius mass">
+    <inertia ixx="${0.4 * mass * radius * radius}" ixy="0.0" ixz="0.0"
+             iyy="${0.4 * mass * radius * radius}" iyz="0.0"
+             izz="${0.4 * mass * radius * radius}" />
+  </xacro:macro>
 </robot>
