Commit message: less damping

File: KUKA_Task/ros_ws/src/iiwa_stack_examples/iiwa_tool/iiwa_tool_description/urdf/tool_pendulum.xacro (robot description, xacro)
@@ -11,5 +11,5 @@
   <xacro:property name="link_offset" value="0 0 ${link_length}" />
   <xacro:property name="link_radius" value="0.0015" />
-  <xacro:property name="joint_damping" value="0.00001" />
+  <xacro:property name="joint_damping" value="0.0000001" />
   <xacro:property name="joint_friction" value="0" />
   <xacro:property name="ball_mass" value="0.2" />

Commit message: better sim, better ode physics

File: KUKA_Task/ros_ws/src/iiwa_stack_examples/iiwa_tool/iiwa_tool_description/urdf/tool_pendulum.xacro (robot description, xacro)
@@ -4,5 +4,5 @@
   <xacro:include filename="$(find iiwa_description)/urdf/utilities.xacro" />
   <!-- Tool properties -->
-  <xacro:property name="tool_mass" value="1" /> <!-- Mass of string -->
+  <xacro:property name="tool_mass" value="0.02" /> <!-- Mass of string -->
   <xacro:property name="tool_length" value="0.24" /> <!-- Length of string -->
   <xacro:property name="num_links" value="10" />
@@ -11,7 +11,7 @@
   <xacro:property name="link_offset" value="0 0 ${link_length}" />
   <xacro:property name="link_radius" value="0.0015" />
-  <xacro:property name="joint_damping" value="0.0000001" />
-  <xacro:property name="joint_friction" value="0" />
-  <xacro:property name="ball_mass" value="0.2" />
+  <xacro:property name="joint_damping" value="0.0001" />
+  <xacro:property name="joint_friction" value="0.01" />
+  <xacro:property name="ball_mass" value="0.02" />
   <xacro:property name="ball_radius" value="${link_radius*10}" />
   <xacro:macro name="tool_pendulum" params="parent *origin">
@@ -53,5 +53,5 @@
       <limit lower="${-90 * PI / 180}" upper="${90 * PI / 180}"
              effort="0" velocity="0" />
-      <dynamics damping="${joint_damping}"/>
+      <dynamics damping="0.001"/>
       <dynamics friction="${joint_friction}"/>
     </joint>

Commit message: physics improvement

File: KUKA_Task/ros_ws/src/iiwa_stack_examples/iiwa_tool/iiwa_tool_description/urdf/tool_pendulum.xacro (robot description, xacro)
@@ -4,5 +4,5 @@
   <xacro:include filename="$(find iiwa_description)/urdf/utilities.xacro" />
   <!-- Tool properties -->
-  <xacro:property name="tool_mass" value="0.02" /> <!-- Mass of string -->
+  <xacro:property name="tool_mass" value="0.025" /> <!-- Mass of string -->
   <xacro:property name="tool_length" value="0.24" /> <!-- Length of string -->
   <xacro:property name="num_links" value="10" />

Commit message: tracking ball position

File: KUKA_Task/ros_ws/src/iiwa_stack_examples/iiwa_tool/iiwa_tool_description/urdf/tool_pendulum.xacro (robot description, xacro)
@@ -49,5 +49,5 @@
       <parent link="tool_link_dummy" />
       <child link = "tool_link_${num_links}" />
-      <origin xyz="0 0 0" rpy="0 0 0" />
+      <origin xyz="0 0 0" rpy="0 ${PI/3} 0" />
       <axis xyz="0 1 0"/> <!-- Only rotate in the y axis i.e. in the x-z plane -->
       <limit lower="${-90 * PI / 180}" upper="${90 * PI / 180}"

File: KUKA_Task/ros_ws/src/iiwa_stack_fishing/iiwa_description/urdf/iiwa.gazebo.xacro (robot description, xacro)
@@ -5,4 +5,13 @@
     <gazebo reference="${robot_name}_joint_7">
       <provideFeedback>true</provideFeedback>
+    </gazebo>
+    <!-- Ball 3-D state ground truth -->
+    <gazebo>
+      <plugin name="Ball_3D_state" filename="libgazebo_ros_p3d.so">
+        <frameName>world</frameName>
+        <bodyName>tool_link_0</bodyName>
+        <topicName>odom/ball</topicName>
+        <updateRate>50.0</updateRate>
+      </plugin>
     </gazebo>
     <!-- The ft_sensor plugin -->

File: KUKA_Task/ros_ws/src/iiwa_stack_fishing/iiwa_description/urdf/iiwa7.xacro (robot description, xacro)
@@ -221,5 +221,5 @@
       <parent link="${robot_name}_link_5"/>
       <child link="${robot_name}_link_6"/>
-      <origin xyz="0 0.06070 0.19" rpy="${PI / 2} ${-PI / 3} 0"/>
+      <origin xyz="0 0.06070 0.19" rpy="${PI / 2} ${-PI / 2} 0"/>
       <axis xyz="0 0 1"/>
       <limit lower="${-120 * PI / 180}" upper="${120 * PI / 180}"
