Commit message: Avishek lunar

File: KUKA_Task/ros_ws/src/iiwa_stack_fishing/iiwa_description/urdf/iiwa7.xacro (robot description, xacro)
@@ -87,5 +87,6 @@
       <origin xyz="0 0 0.19" rpy="${PI / 2}   ${-PI / 3} ${PI}"/>
       <axis xyz="0 0 1"/>
-      <limit lower="${-120 * PI / 180}" upper="${120 * PI / 180}"
+      <!-- <limit lower="${-120 * PI / 180}" upper="${120 * PI / 180}" -->
+      <limit lower="${-60 * PI / 180}" upper="${30 * PI / 180}"
              effort="${max_effort}" velocity="${max_velocity}" />
       <safety_controller soft_lower_limit="${-118 * PI / 180}"
@@ -155,5 +156,6 @@
       <origin xyz="0 0 0.19" rpy="${PI / 2} ${PI / 6} 0"/>
       <axis xyz="0 0 1"/>
-      <limit lower="${-120 * PI / 180}" upper="${120 * PI / 180}"
+      <!-- <limit lower="${-120 * PI / 180}" upper="${120 * PI / 180}" -->
+      <limit lower="${-60 * PI / 180}" upper="${30 * PI / 180}"
              effort="${max_effort}" velocity="${max_velocity}" />
       <safety_controller soft_lower_limit="${-118 * PI / 180}"

Commit message: Better sim and learn tpolicy

File: KUKA_Task/ros_ws/src/iiwa_stack_fishing/iiwa_description/urdf/iiwa7.xacro (robot description, xacro)
@@ -85,8 +85,8 @@
       <parent link="${robot_name}_link_1"/>
       <child link="${robot_name}_link_2"/>
-      <origin xyz="0 0 0.19" rpy="${PI / 2}   ${-PI / 3} ${PI}"/>
+      <origin xyz="0 0 0.19" rpy="${PI / 2}   ${-40 * PI / 180} ${PI}"/>
       <axis xyz="0 0 1"/>
       <!-- <limit lower="${-120 * PI / 180}" upper="${120 * PI / 180}" -->
-      <limit lower="${-60 * PI / 180}" upper="${30 * PI / 180}"
+      <limit lower="${-40 * PI / 180}" upper="${50 * PI / 180}"
              effort="${max_effort}" velocity="${max_velocity}" />
       <safety_controller soft_lower_limit="${-118 * PI / 180}"

Commit message: improved ball position

File: KUKA_Task/ros_ws/src/iiwa_stack_fishing/iiwa_description/urdf/iiwa7.xacro (robot description, xacro)
@@ -85,9 +85,9 @@
       <parent link="${robot_name}_link_1"/>
       <child link="${robot_name}_link_2"/>
-      <origin xyz="0 0 0.19" rpy="${PI / 2}   ${-40 * PI / 180} ${PI}"/>
-      <axis xyz="0 0 1"/>
-      <!-- <limit lower="${-120 * PI / 180}" upper="${120 * PI / 180}" -->
-      <limit lower="${-40 * PI / 180}" upper="${50 * PI / 180}"
-             effort="${max_effort}" velocity="${max_velocity}" />
+      <origin xyz="0 0 0.19" rpy="${PI / 2}   ${-45 * PI / 180} ${PI}"/>
+      <axis xyz="0 0 1"/>
+      <limit lower="${-120 * PI / 180}" upper="${120 * PI / 180}"
+              effort="${max_effort}" velocity="${max_velocity}" />
+      <!-- <limit lower="${-40 * PI / 180}" upper="${50 * PI / 180}" -->
       <safety_controller soft_lower_limit="${-118 * PI / 180}"
                          soft_upper_limit="${118 * PI / 180}"
@@ -154,9 +154,9 @@
       <parent link="${robot_name}_link_3"/>
       <child link="${robot_name}_link_4"/>
-      <origin xyz="0 0 0.19" rpy="${PI / 2} ${PI / 6} 0"/>
-      <axis xyz="0 0 1"/>
-      <!-- <limit lower="${-120 * PI / 180}" upper="${120 * PI / 180}" -->
-      <limit lower="${-60 * PI / 180}" upper="${30 * PI / 180}"
-             effort="${max_effort}" velocity="${max_velocity}" />
+      <origin xyz="0 0 0.19" rpy="${PI / 2} ${PI / 4} 0"/>
+      <axis xyz="0 0 1"/>
+      <limit lower="${-120 * PI / 180}" upper="${120 * PI / 180}"
+              effort="${max_effort}" velocity="${max_velocity}" />
+      <!-- <limit lower="${-60 * PI / 180}" upper="${30 * PI / 180}" -->
       <safety_controller soft_lower_limit="${-118 * PI / 180}"
                          soft_upper_limit="${118 * PI / 180}"
